File: usb-audio-interface.kicad_pcb (KiCad board)
At the start: 2 copper layers, 25 parts, among them IC1 PCM2906C, J1 USB_C_Receptacle_USB2.0_14P, J2 Conn_Coaxial_x2, J3 Conn_Coaxial, J4 Conn_Coaxial_x2, J5 Conn_Coaxial, Y1 12MHz

Commit message: finish pcb
Parts:
- Y1: footprint Crystal:Crystal_SMD_HC49-SD_HandSoldering -> Crystal:Crystal_SMD_HC49-SD
- moved C3 85.0 mm to (158.5, 74.8), turned to -90 degrees
- moved C6 81.5 mm to (158.5, 58.5), turned to 90 degrees
- moved J2 74.1 mm to (166.5, 45.5), turned to 180 degrees
- moved C4 72.6 mm to (148.5, 74.8), turned to -90 degrees
- moved C5 70.2 mm to (148.5, 58.5), turned to 90 degrees
- moved J4 64.2 mm to (151.5, 87.6)
- moved J3 52.8 mm to (138.5, 48.6), turned to 180 degrees
- moved Y1 47.0 mm to (138.5, 66.5), turned to -90 degrees
- moved C1 36.9 mm to (170.0, 72.5)
- moved J5 35.6 mm to (138.5, 84.5)
- moved C2 33.6 mm to (147.0, 70.5)
- moved C8 33.1 mm to (142.0, 61.5), turned to 90 degrees
- moved C7 28.8 mm to (142.0, 71.5), turned to -90 degrees
- moved R5 5.79 mm to (135.0, 66.5), turned to 90 degrees
- moved R2 5.43 mm to (161.6, 71.0), turned to 180 degrees
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Routing:
- net GND: track 0.00 -> 214.3 mm
- net VBUS: track 0.00 -> 30.2 mm
- net /DOUT: track 0.00 -> 27.8 mm, vias 0 -> 1
- net /DIN: track 0.00 -> 27.2 mm, vias 0 -> 1
- net VDD: track 0.00 -> 21.0 mm, vias 0 -> 2
- net /XTI: track 0.00 -> 18.5 mm
- net /VINR: track 0.00 -> 18.0 mm
- net /XTO: track 0.00 -> 17.8 mm
- net /VINL: track 0.00 -> 15.2 mm
- net Net-(J2-IN2): track 0.00 -> 14.6 mm
- net Net-(J1-D+-PadA6): track 0.00 -> 12.0 mm
- net /VOUTR: track 0.00 -> 11.4 mm
- net Net-(J2-IN1): track 0.00 -> 9.15 mm
- net Net-(J1-D--PadA7): track 0.00 -> 8.90 mm
- net /D-: track 0.00 -> 7.56 mm
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- added copper zone on B.Cu, net GND
- added copper zone on F.Cu, net GND
Other:
- board outline added: 41.5 x 56 mm
- rule pad_to_mask_clearance: 0 -> 0.0508
