File: usb-audio-interface.kicad_sch (KiCad schematic)
At the start: 21 parts, among them IC1 PCM2906CDBR, J1 USB_C_Receptacle_USB2.0_14P, J2 Conn_Coaxial_x2, J3 Conn_Coaxial, Y1 12MHz

Commit message: Update schematic and start on footprints
Parts:
- added C3, C4: 820uF, symbol Device:C_Polarized_Small
- added J4: Conn_Coaxial_x2, symbol Connector:Conn_Coaxial_x2
- added J5: Conn_Coaxial, symbol Connector:Conn_Coaxial
- C1: renamed from C20; footprint Capacitor_THT:C_Rect_L7.0mm_W2.0mm_P5.00mm -> Capacitor_SMD:C_0201_0603Metric_Pad0.64x0.40mm_HandSolder
- C10: renamed from C6; footprint (none) -> Capacitor_SMD:C_0201_0603Metric_Pad0.64x0.40mm_HandSolder
- C11: renamed from C7; footprint (none) -> Capacitor_SMD:C_0201_0603Metric_Pad0.64x0.40mm_HandSolder
- C2: footprint (none) -> Capacitor_SMD:C_0201_0603Metric_Pad0.64x0.40mm_HandSolder
- C9: renamed from C5; footprint (none) -> Capacitor_SMD:C_0201_0603Metric_Pad0.64x0.40mm_HandSolder
- IC1: footprint SOP65P780X200-28N -> Package_SO:Texas_PWP0028V_TSSOP-28-1EP_4.4x9.7mm_P0.65mm_EP3.4x9.7mm_Mask2.94x5.62mm
- R1, R2, R3: footprint Resistor_THT:R_Axial_DIN0207_L6.3mm_D2.5mm_P10.16mm_Horizontal -> Resistor_SMD:R_0201_0603Metric_Pad0.64x0.40mm_HandSolder
- R4, R5: footprint (none) -> Resistor_SMD:R_0201_0603Metric_Pad0.64x0.40mm_HandSolder
- renumbered C8 to C12, C9 to C13, C1 to C5, C10 to C6, C3 to C7, C4 to C8
Connections:
- net D+: no longer R4.1
- net DIN: now also J5.1 (In)
- net GND: now also J4.3 (EXT), J5.2 (Ext)
- net VINL: now also C3.1
- net VINR: now also C4.1
- net at J1.A6 (D+), J1.B6 (D+), R3.1: now also R4.1
- new net: C3.2, J4.1 (IN1)
- new net: C4.2, J4.2 (IN2)
Other:
- note added: "Audio inputs"
- note added: "Audio outputs"
- moved on the sheet: C10, C11, C12, C13, C2, C5, C6, C7, C8, C9, J2, J3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

Commit message: finish schematic
Parts:
- C1, C10, C11, C2, C9: footprint Capacitor_SMD:C_0201_0603Metric_Pad0.64x0.40mm_HandSolder -> Capacitor_SMD:C_0603_1608Metric_Pad1.08x0.95mm_HandSolder; Manufacturer_Name (none) -> Samsung Electro-Mechanics; Manufacturer_Part_Number (none) -> CL10A105KQ8NNNC
- C12, C13: footprint (none) -> Capacitor_SMD:C_0805_2012Metric_Pad1.18x1.45mm_HandSolder; symbol Device:C_Polarized_Small -> Device:C_Small; Manufacturer_Name (none) -> Samsung Electro-Mechanics; Manufacturer_Part_Number (none) -> CL21A106KOQNNNG
- C3, C4, C5, C6: footprint (none) -> Capacitor_THT:CP_Radial_D8.0mm_P3.50mm; Manufacturer_Name (none) -> Rubycon; Manufacturer_Part_Number (none) -> 6.3ZLH820MEFC8X11.5
- C7, C8: value C_Small -> 25pF; footprint (none) -> Capacitor_SMD:C_0603_1608Metric_Pad1.08x0.95mm_HandSolder; Manufacturer_Name (none) -> Walsin; Manufacturer_Part_Number (none) -> 0603N250K500CT
- IC1: footprint Package_SO:Texas_PWP0028V_TSSOP-28-1EP_4.4x9.7mm_P0.65mm_EP3.4x9.7mm_Mask2.94x5.62mm -> Package_SO:SSOP-28_5.3x10.2mm_P0.65mm
- J1: Manufacturer_Name (none) -> GCT; Manufacturer_Part_Number (none) -> USB4105-GF-A-120
- J2, J4: footprint (none) -> RCA jacks:PJRAN2X1U01AUX; Manufacturer_Name (none) -> Switchcraft; Manufacturer_Part_Number (none) -> PJRAN2X1U01AUX
- J3, J5: footprint (none) -> RCA jacks:1560099E; Manufacturer_Name (none) -> Kobiconn; Manufacturer_Part_Number (none) -> 156-0099-E
- R1: footprint Resistor_SMD:R_0201_0603Metric_Pad0.64x0.40mm_HandSolder -> Resistor_SMD:R_0603_1608Metric_Pad0.98x0.95mm_HandSolder; Manufacturer_Name (none) -> Kamaya; Manufacturer_Part_Number (none) -> RMC1/16-512JTP
- R2, R3: footprint Resistor_SMD:R_0201_0603Metric_Pad0.64x0.40mm_HandSolder -> Resistor_SMD:R_0603_1608Metric_Pad0.98x0.95mm_HandSolder; Manufacturer_Name (none) -> YAGEO; Manufacturer_Part_Number (none) -> RT0603DRD0722RL
- R4: footprint Resistor_SMD:R_0201_0603Metric_Pad0.64x0.40mm_HandSolder -> Resistor_SMD:R_0603_1608Metric_Pad0.98x0.95mm_HandSolder; Manufacturer_Name (none) -> TE Connectivity / Holsworthy; Manufacturer_Part_Number (none) -> CRGCQ0603F1K5
- R5: footprint Resistor_SMD:R_0201_0603Metric_Pad0.64x0.40mm_HandSolder -> Resistor_SMD:R_0603_1608Metric_Pad0.98x0.95mm_HandSolder; Manufacturer_Name (none) -> KOA Speer; Manufacturer_Part_Number (none) -> RK73B1JTTDD105J
- Y1: footprint (none) -> Crystal:Crystal_SMD_HC49-SD_HandSoldering; Manufacturer_Name (none) -> ABRACON; Manufacturer_Part_Number (none) -> ABLS-12.000MHz-B4H-T

Commit message: finish pcb
Parts:
- IC1: value PCM2906CDBR -> PCM2906C
- Y1: footprint Crystal:Crystal_SMD_HC49-SD_HandSoldering -> Crystal:Crystal_SMD_HC49-SD
Changed lines of the file:
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@@
 			)
 		)
-		(property "Value" "PCM2906CDBR"
+		(property "Value" "PCM2906C"
 			(at 135.382 87.63 0)
 			(effects
@@
 			)
 		)
-		(property "Footprint" "Crystal:Crystal_SMD_HC49-SD_HandSoldering"
+		(property "Footprint" "Crystal:Crystal_SMD_HC49-SD"
 			(at 236.22 90.17 0)
 			(effects

Commit message: update bom
Parts:
- C7, C8: Manufacturer_Name Walsin -> YAGEO; Manufacturer_Part_Number 0603N250K500CT -> CC0603JRNPO9BN250
Changed lines of the file:
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@@
 	(label "D-"
 		(at 105.41 128.27 0)
-		(fields_autoplaced yes)
 		(effects
 			(font
@@
 	(label "XTI"
 		(at 210.82 86.36 0)
-		(fields_autoplaced yes)
 		(effects
 			(font
@@
 	(label "DIN"
 		(at 53.34 116.84 180)
-		(fields_autoplaced yes)
 		(effects
 			(font
@@
 	(label "VINR"
 		(at 53.34 99.06 180)
-		(fields_autoplaced yes)
 		(effects
 			(font
@@
 	(label "XTI"
 		(at 161.29 104.14 180)
-		(fields_autoplaced yes)
 		(effects
 			(font
@@
 	(label "VCCP1I"
 		(at 161.29 118.11 180)
-		(fields_autoplaced yes)
 		(effects
 			(font
@@
 	(label "XTO"
 		(at 210.82 93.98 0)
-		(fields_autoplaced yes)
 		(effects
 			(font
@@
 	(label "VCCP2I"
 		(at 234.95 128.27 0)
-		(fields_autoplaced yes)
 		(effects
 			(font
@@
 	(label "XTO"
 		(at 161.29 106.68 180)
-		(fields_autoplaced yes)
 		(effects
 			(font
@@
 	(label "VOUTL"
 		(at 224.79 30.48 0)
-		(fields_autoplaced yes)
 		(effects
 			(font
@@
 	(label "VOUTL"
 		(at 161.29 91.44 180)
-		(fields_autoplaced yes)
 		(effects
 			(font
@@
 	(label "VCCCI"
 		(at 161.29 113.03 180)
-		(fields_autoplaced yes)
 		(effects
 			(font
@@
 	(label "DOUT"
 		(at 224.79 57.15 0)
-		(fields_autoplaced yes)
 		(effects
 			(font
@@
 	(label "VCCP2I"
 		(at 161.29 120.65 180)
-		(fields_autoplaced yes)
 		(effects
 			(font
@@
 	(label "DOUT"
 		(at 161.29 99.06 180)
-		(fields_autoplaced yes)
 		(effects
 			(font
@@
 	(label "VCOM"
 		(at 161.29 115.57 180)
-		(fields_autoplaced yes)
 		(effects
 			(font
@@
 	(label "D-"
 		(at 69.85 38.1 180)
-		(fields_autoplaced yes)
 		(effects
 			(font
@@
 	(label "DIN"
 		(at 105.41 99.06 0)
-		(fields_autoplaced yes)
 		(effects
 			(font
@@
 	(label "VOUTR"
 		(at 161.29 93.98 180)
-		(fields_autoplaced yes)
 		(effects
 			(font
@@
 	(label "VCOM"
 		(at 234.95 158.75 0)
-		(fields_autoplaced yes)
 		(effects
 			(font
@@
 	(label "VINR"
 		(at 105.41 93.98 0)
-		(fields_autoplaced yes)
 		(effects
 			(font
@@
 	(label "D+"
 		(at 105.41 125.73 0)
-		(fields_autoplaced yes)
 		(effects
 			(font
@@
 	(label "VCCP1I"
 		(at 234.95 118.11 0)
-		(fields_autoplaced yes)
 		(effects
 			(font
@@
 	(label "VINL"
 		(at 53.34 93.98 180)
-		(fields_autoplaced yes)
 		(effects
 			(font
@@
 	(label "VOUTR"
 		(at 224.79 35.56 0)
-		(fields_autoplaced yes)
 		(effects
 			(font
@@
 	(label "VCCCI"
 		(at 234.95 148.59 0)
-		(fields_autoplaced yes)
 		(effects
 			(font
@@
 	(label "VCCXI"
 		(at 234.95 138.43 0)
-		(fields_autoplaced yes)
 		(effects
 			(font
@@
 	(label "VINL"
 		(at 105.41 91.44 0)
-		(fields_autoplaced yes)
 		(effects
 			(font
@@
 	(label "D+"
 		(at 69.85 43.18 180)
-		(fields_autoplaced yes)
 		(effects
 			(font
@@
 	(label "VCCXI"
 		(at 161.29 123.19 180)
-		(fields_autoplaced yes)
 		(effects
 			(font
@@
 			)
 		)
-		(property "Datasheet" "https://www.mouser.com/datasheet/2/210/WTC_MLCC_General_Purpose-1534899.pdf"
+		(property "Datasheet" "https://www.mouser.com/datasheet/2/447/upy_np0x7r_mv_100_to_630v-3461223.pdf"
 			(at 251.46 86.36 0)
 			(effects
@@
 			)
 		)
-		(property "Manufacturer_Name" "Walsin"
+		(property "Manufacturer_Name" "YAGEO"
 			(at 251.46 86.36 0)
 			(effects
@@
 			)
 		)
-		(property "Manufacturer_Part_Number" "0603N250K500CT "
+		(property "Manufacturer_Part_Number" "CC0603JRNPO9BN250"
 			(at 251.46 86.36 0)
 			(effects
@@
 			)
 		)
-		(property "Datasheet" "https://www.mouser.com/datasheet/2/210/WTC_MLCC_General_Purpose-1534899.pdf"
+		(property "Datasheet" "https://www.mouser.com/datasheet/2/447/upy_np0x7r_mv_100_to_630v-3461223.pdf"
 			(at 251.46 93.98 0)
 			(effects
@@
 			)
 		)
-		(property "Manufacturer_Name" "Walsin"
+		(property "Manufacturer_Name" "YAGEO"
 			(at 251.46 93.98 0)
 			(effects
@@
 			)
 		)
-		(property "Manufacturer_Part_Number" "0603N250K500CT "
+		(property "Manufacturer_Part_Number" "CC0603JRNPO9BN250"
 			(at 251.46 93.98 0)
 			(effects
